Commit message: Add working gazebo thruster plugin (values need to be adjusted)

File: catkin_ws/src/auv_description/urdf/bradbury.urdf.xacro (robot description, xacro)
@@ -13,10 +13,10 @@
   <xacro:property name="frame_height" value="0.27" />
   <!-- MADE UP VALUE -->
-  <xacro:property name="frame_mass" value="4" />
+  <xacro:property name="frame_mass" value="1" />
   <!-- Main Hull -->
   <xacro:property name="main_hull_radius" value="0.125" />
   <xacro:property name="main_hull_length" value="0.52" />
   <!-- MADE UP VALUE -->
-  <xacro:property name="main_hull_mass" value="2" />
+  <xacro:property name="main_hull_mass" value="1.0" />
   <!-- Battery PV -->
   <xacro:property name="battery_radius" value="0.1" />
@@ -48,5 +48,5 @@
     </link>
     <joint name="base_to_${prefix}_thruster" type="fixed">
-      <parent link="base_link"/>
+      <parent link="frame"/>
       <child link="${prefix}_thruster"/>
       <origin rpy ="${roll} ${pitch} ${yaw}" xyz="${x} ${y} ${z}"/>
@@ -55,4 +55,10 @@
   <!-- Frame - base_link is the center of the frame, and center of surger thrusters in z. -->
   <link name="frame">
+    <visual>
+      <origin rpy="${pi/2} 0 ${pi}" xyz="0.41552 -0.1554 -0.2159"/>
+      <geometry>
+        <mesh filename="package://auv_description/meshes/frame.stl" scale="0.01 0.01 0.01"/>
+      </geometry>
+    </visual>
     <collision>
       <origin rpy="0 0 0" xyz="0 0 0"/>
@@ -71,10 +77,4 @@
   </link>
   <link name="base_link">
-    <visual>
-      <origin rpy="${pi/2} 0 ${pi}" xyz="0.41552 -0.1554 -0.2159"/>
-      <geometry>
-        <mesh filename="package://auv_description/meshes/frame.stl" scale="0.01 0.01 0.01"/>
-      </geometry>
-    </visual>
   </link>
   <!-- Main PV -->
@@ -132,5 +132,5 @@
   <!-- MAIN HULL TO FRAME JOINT -->
   <joint name="base_to_main_hull" type="fixed">
-    <parent link="base_link"/>
+    <parent link="frame"/>
     <child link="main_hull"/>
     <origin rpy="0 0 0" xyz="0 0 0.1547"/>
@@ -138,5 +138,5 @@
   <!-- BATTERY TO FRAME JOINT -->
   <joint name="base_to_battery" type="fixed">
-    <parent link="base_link"/>
+    <parent link="frame"/>
     <child link="battery"/>
     <origin rpy="0 0 0" xyz="0.2614 0 -0.1038"/>
@@ -151,27 +151,12 @@
   <xacro:thruster prefix="bow_sway" yaw="${pi/2}" roll="0" pitch="0" x="0.465" y="0" z="${sway_depth}"/>
   <xacro:thruster prefix="stern_sway" yaw="${-pi/2}" roll="0" pitch="0" x="-0.465" y="0" z="${sway_depth}"/>
-  <!-- GAZEBO MACROS -->
-  <xacro:macro name="thruster_gazebo" params="prefix">
-      <gazebo reference="${prefix}_thruster">
-          <material>Gazebo/Red</material>
-          <selfCollide>false</selfCollide>
-          <!--dampingFactor>0.0001</dampingFactor-->
-      </gazebo>
-      <gazebo reference="base_to_${prefix}_thruster">
-          <!-- <implicitSpringDamper>true</implicitSpringDamper> -->
-      </gazebo>
-  </xacro:macro>
   <!-- GAZEBO SPECIFIC SETTINGS -->
   <gazebo reference="base_link">
+      <selfCollide>false</selfCollide>
+      <static>false</static>
+  </gazebo>
+  <gazebo reference="frame">
       <material>Gazebo/Grey</material>
       <selfCollide>false</selfCollide>
   </gazebo>
-  <xacro:thruster_gazebo prefix="surge_port"/>
-  <xacro:thruster_gazebo prefix="starboard_surge"/>
-  <xacro:thruster_gazebo prefix="port_bow_heave"/>
-  <xacro:thruster_gazebo prefix="port_stern_heave"/>
-  <xacro:thruster_gazebo prefix="starboard_bow_heave"/>
-  <xacro:thruster_gazebo prefix="starboard_stern_heave"/>
-  <xacro:thruster_gazebo prefix="bow_sway"/>
-  <xacro:thruster_gazebo prefix="stern_sway"/>
 </robot>

File: catkin_ws/src/auv_gazebo/urdf/auv_plugins.urdf.xacro (robot description, xacro)
@@ -1,7 +1,30 @@
 <?xml version="1.0"?>
-<robot xmlns:xacro="http://ros.org/wiki/xacro">
-  <gazebo>
+<robot xmlns:xacro="http://ros.org/wiki/xacro" name="bradbury">
+   <gazebo>
     <plugin name="thruster_plugin" filename="libthruster_plugin.so">
     </plugin>
   </gazebo>
+  <gazebo>
+    <plugin name="lifting_surface" filename="libLiftDragPlugin.so">
+      <link_name>base_link</link_name>
+      <air_density>1000</air_density>
+      <cla>1.25</cla>  <!-- 1.2535816618911175 -->
+      <cla_stall>-85.0</cla_stall>  <!-- 1.4326647564469914 -->
+      <cda>0</cda>
+      <cda_stall>85.0</cda_stall>
+      <alpha_stall>0</alpha_stall>
+      <a0>0</a0>
+      <area>0.5</area>
+      <upward>0 0 -1</upward>
+      <forward>1 0 0</forward>
+      <cp>0 0 0</cp>
+    </plugin>
+  </gazebo>
+  <gazebo>
+    <plugin name="buoyancy_plugin" filename="libBuoyancyPlugin.so">
+      <link name="base_link">
+      </link>
+      <fluid_density>1000</fluid_density>
+    </plugin>
+  </gazebo>
 </robot>

Commit message: Add comments

File: catkin_ws/src/auv_description/urdf/bradbury.urdf.xacro (robot description, xacro)
@@ -18,5 +18,5 @@
   <xacro:property name="main_hull_length" value="0.52" />
   <!-- MADE UP VALUE -->
-  <xacro:property name="main_hull_mass" value="1.0" />
+  <xacro:property name="main_hull_mass" value="20.0" />
   <!-- Battery PV -->
   <xacro:property name="battery_radius" value="0.1" />

Commit message: Add robot to base_link for backwards compatibility

File: catkin_ws/src/auv_description/urdf/bradbury.urdf.xacro (robot description, xacro)
@@ -78,4 +78,7 @@
   <link name="base_link">
   </link>
+  <!-- This is needed for backwards compatibility only. -->
+  <link name="robot">
+  </link>
   <!-- Main PV -->
   <link name="main_hull">
@@ -125,4 +128,10 @@
     </inertial>
   </link>
+  <!-- This is needed for backwards compatibility only. -->
+  <joint name="base_to_robot" type="fixed">
+    <parent link="robot"/>
+    <child link="base_link"/>
+    <origin rpy="0 0 0" xyz="0 0 0"/>
+  </joint>
   <joint name="base_to_frame" type="fixed">
     <parent link="base_link"/>
