Commit message: Pack auv_desc/viz/gazebo into sim package

File: catkin_ws/src/simulation/models/urdf/bradbury.urdf.xacro (robot description, xacro)
@@ -29,5 +29,5 @@
         <origin rpy ="0 ${pi/2} 0" xyz="0 0 0"/>
         <geometry>
-          <mesh filename="package://auv_description/meshes/thruster.stl" scale="0.01 0.01 0.01"/>
+          <mesh filename="package://simulation/models//meshes/thruster.stl" scale="0.01 0.01 0.01"/>
         </geometry>
       </visual>
@@ -58,5 +58,5 @@
       <origin rpy="${pi/2} 0 ${pi}" xyz="0.41552 -0.1554 -0.2159"/>
       <geometry>
-        <mesh filename="package://auv_description/meshes/frame.stl" scale="0.01 0.01 0.01"/>
+        <mesh filename="package://simulation/models//meshes/frame.stl" scale="0.01 0.01 0.01"/>
       </geometry>
     </visual>
@@ -86,5 +86,5 @@
       <origin rpy="${pi/2} 0 ${pi/2}" xyz="-0.2594 0 0"/>
       <geometry>
-        <mesh filename="package://auv_description/meshes/main_hull.stl" scale="0.01 0.01 0.01"/>
+        <mesh filename="package://simulation/models//meshes/main_hull.stl" scale="0.01 0.01 0.01"/>
       </geometry>
     </visual>
@@ -110,5 +110,5 @@
       <origin rpy="${pi/2} 0 0" xyz="0 0.1572 0"/>
       <geometry>
-        <mesh filename="package://auv_description/meshes/battery.stl" scale="0.01 0.01 0.01"/>
+        <mesh filename="package://simulation/models//meshes/battery.stl" scale="0.01 0.01 0.01"/>
       </geometry>
     </visual>
